File: RSAO232/RSAO232.kicad_sch (KiCad schematic)
At the start: 20 parts, among them J1 DE9_Receptacle_MountingHoles, U1 SC16IS740, U2 MAX3232, Y1 1.8432 MHz

Commit message: Almost finished schematic and layout, probably need a bit more bulk capacitance
Parts:
- added C7, C8: 100n, Capacitor_SMD:C_0603_1608Metric_Pad1.08x0.95mm_HandSolder, symbol Device:C
- added JP1: IRQ, Jumper:SolderJumper-2_P1.3mm_Open_RoundedPad1.0x1.5mm, symbol Jumper:SolderJumper_2_Open
- added X1: Simple_Addon_v2, Simple_Addon_v2:Simple_Addon_v2-SAO-2x3-SMD, symbol Simple_Addon_v2:Simple_Addon_v2
- C1, C2, C3, C4, C5, C6: footprint (none) -> Capacitor_SMD:C_0603_1608Metric_Pad1.08x0.95mm_HandSolder
- J1: footprint (none) -> Connector_Dsub:DSUB-9_Female_Vertical_P2.77x2.84mm_MountingHoles
- R1, R10, R2, R3, R4, R5, R6, R7, R8, R9: footprint (none) -> Resistor_SMD:R_0603_1608Metric_Pad0.98x0.95mm_HandSolder
- U2: footprint (none) -> Package_SO:SOIC-16_3.9x9.9mm_P1.27mm
- Y1: footprint (none) -> Crystal:Crystal_SMD_HC49-SD
Connections:
- net +3V3: now also C7.1, C8.1, X1.1 (VCC)
- net GND: now also C7.2, C8.2, X1.2 (GND)
- net RS232_IRQ: now also JP1.1 (A)
- net SCL: now also X1.4 (SCL)
- net SDA: now also X1.3 (SDA)
- new net: JP1.2 (B), X1.5 (GPIO1)
- no-connect marks 5 -> 6
